File: Hardware/SHTC3 Breakout.brd (EAGLE design)
At the start: 25.4 x 25.4 mm, 33 parts, among them J3 PTH, U1 SHTC3

Commit message: Decrease via size. Change Qwiic logo.
Parts:
- removed U$29: (no value), Labels:QWIIC-LOGO-MEDIUM
- added U$11, U$12: (no value), SparkFun-Aesthetics:QWIIC_5.5MM
Other:
- board text added: "x02"
- board text removed: "X01"
