File: Hardware/Production/SHTC3 Breakout-Panel.brd (EAGLE design)
At the start: 0 parts

Commit message: Correcting HW Version
Looks like release version wasn't commited.  Updating.
Parts:
- added C1, C2, C3, C4, C5, C6, C7, C8, C9: 0.1uF, SparkFun-Capacitors:0603
- added D1, D2, D3, D4, D5, D6, D7, D8, D9: RED, SparkFun-LED:LED-0603
- added E$1, E$2: (no value), SparkFun-Aesthetics:FIDUCIAL-1X2
- added E$3: (no value), SparkFun-Retired:FIDUCIAL-1.5X3
- added J1, J10, J12, J13, J15, J16, J18, J19, J2, J21, J22, J24, J25, J27, J4, J6, J7, J9: (no value), SparkFun-Connectors:1X04_1MM_RA
- added J11, J14, J17, J20, J23, J26, J3, J5, J8: PTH, SparkX:1X04_NO_SILK
- added JP1, JP10, JP11, JP12, JP13, JP17, JP18, JP19, JP2, JP20, JP24, JP25, JP26, JP27, JP31, JP32, JP33, JP34, JP38, JP39, JP40, JP41, JP45, JP46, JP47, JP48, JP5, JP52, JP53, JP54, JP55, JP59, JP6, JP60, JP61, JP62: FIDUCIALUFIDUCIAL, SparkFun:MICRO-FIDUCIAL
- added JP14, JP21, JP28, JP35, JP42, JP49, JP56, JP63, JP7: JUMPER-SMT_3_2-NC_TRACE_SILK, SparkFun-Jumpers:SMT-JUMPER_3_2-NC_TRACE_SILK
- added JP15, JP16, JP22, JP23, JP29, JP3, JP30, JP36, JP37, JP4, JP43, JP44, JP50, JP51, JP57, JP58, JP8, JP9: STAND-OFF, SparkFun:STAND-OFF
- added LOGO1, LOGO2, LOGO3, LOGO4, LOGO5, LOGO6, LOGO7, LOGO8, LOGO9: OSHW-LOGOMINI, SparkFun-Aesthetics:OSHW-LOGO-MINI
- added R1, R11, R12, R14, R15, R17, R18, R2, R20, R21, R23, R24, R26, R27, R5, R6, R8, R9: 2.2k, SparkFun-Resistors:0603
- added R10, R13, R16, R19, R22, R25, R3, R4, R7: 1k, SparkFun-Resistors:0603
- added U$1, U$106, U$107, U$11, U$12, U$121, U$122, U$2, U$31, U$32, U$46, U$47, U$61, U$62, U$76, U$77, U$91, U$92: SPARKX-LOGO4, SparkX:SPARKX-MEDIUM
- added U$10, U$101, U$116, U$131, U$23, U$41, U$56, U$71, U$86: (no value), Labels-0_04:(PWR)
- added U$100, U$110, U$115, U$125, U$130, U$15, U$20, U$26, U$35, U$40, U$50, U$55, U$6, U$65, U$70, U$80, U$85, U$95: (no value), Labels-0_04:SCL9
- added U$102, U$117, U$132, U$24, U$29, U$42, U$57, U$72, U$87: (no value), Labels:QWIIC-LOGO-MEDIUM
- added U$103, U$104, U$118, U$119, U$133, U$134, U$25, U$28, U$43, U$44, U$58, U$59, U$7, U$73, U$74, U$8, U$88, U$89: (no value), buzzard_labels:SHTC3_HUMIDITY1
- added U$105, U$120, U$135, U$30, U$45, U$60, U$75, U$9, U$90: (no value), Labels:I_SUPER2_C-()-03
- added U$108, U$113, U$123, U$128, U$13, U$18, U$21, U$33, U$38, U$4, U$48, U$53, U$63, U$68, U$78, U$83, U$93, U$98: (no value), Labels-0_04:3#3V2
- added U$109, U$112, U$124, U$127, U$14, U$17, U$22, U$3, U$34, U$37, U$49, U$52, U$64, U$67, U$79, U$82, U$94, U$97: (no value), Labels-0_04:GND1
- added U$111, U$114, U$126, U$129, U$16, U$19, U$27, U$36, U$39, U$5, U$51, U$54, U$66, U$69, U$81, U$84, U$96, U$99: (no value), Labels-0_04:SDA8
- added U1, U2, U3, U4, U5, U6, U7, U8, U9: SHTC3, SHTC3:SHTC3
Connections:
- new net 3.3V: C1.1, J2.2, J3.2, J4.2, JP7.2, R3.2, U1.1
- new net 3.3V1: C2.1, J1.2, J5.2, J6.2, JP14.2, R4.2, U2.1
- new net 3.3V2: C3.1, J7.2, J8.2, J9.2, JP21.2, R7.2, U3.1
- new net 3.3V3: C4.1, J10.2, J11.2, J12.2, JP28.2, R10.2, U4.1
- new net 3.3V4: C5.1, J13.2, J14.2, J15.2, JP35.2, R13.2, U5.1
- new net 3.3V5: C6.1, J16.2, J17.2, J18.2, JP42.2, R16.2, U6.1
- new net 3.3V6: C7.1, J19.2, J20.2, J21.2, JP49.2, R19.2, U7.1
- new net 3.3V7: C8.1, J22.2, J23.2, J24.2, JP56.2, R22.2, U8.1
- new net 3.3V8: C9.1, J25.2, J26.2, J27.2, JP63.2, R25.2, U9.1
- new net GND: C1.2, D1.C, J2.1, J3.1, J4.1, U1.4, U1.5
- new net GND1: C2.2, D2.C, J1.1, J5.1, J6.1, U2.4, U2.5
- new net GND2: C3.2, D3.C, J7.1, J8.1, J9.1, U3.4, U3.5
- new net GND3: C4.2, D4.C, J10.1, J11.1, J12.1, U4.4, U4.5
- new net GND4: C5.2, D5.C, J13.1, J14.1, J15.1, U5.4, U5.5
- new net GND5: C6.2, D6.C, J16.1, J17.1, J18.1, U6.4, U6.5
- new net GND6: C7.2, D7.C, J19.1, J20.1, J21.1, U7.4, U7.5
- new net GND7: C8.2, D8.C, J22.1, J23.1, J24.1, U8.4, U8.5
- new net GND8: C9.2, D9.C, J25.1, J26.1, J27.1, U9.4, U9.5
- new net N$1: JP7.3, R1.2
- new net N$10: D4.A, R10.1
- new net N$11: JP28.3, R11.2
- new net N$12: JP28.1, R12.2
- new net N$13: D5.A, R13.1
- new net N$14: JP35.3, R14.2
- new net N$15: JP35.1, R15.2
- new net N$16: D6.A, R16.1
- new net N$17: JP42.3, R17.2
- new net N$18: JP42.1, R18.2
- new net N$19: D7.A, R19.1
- new net N$2: JP7.1, R2.2
- new net N$20: JP49.3, R20.2
- new net N$21: JP49.1, R21.2
- new net N$22: D8.A, R22.1
- new net N$23: JP56.3, R23.2
- new net N$24: JP56.1, R24.2
- new net N$25: D9.A, R25.1
- new net N$26: JP63.3, R26.2
- new net N$27: JP63.1, R27.2
- new net N$3: D1.A, R3.1
- new net N$4: D2.A, R4.1
- new net N$5: JP14.3, R5.2
- new net N$6: JP14.1, R6.2
- new net N$7: D3.A, R7.1
- new net N$8: JP21.3, R8.2
- new net N$9: JP21.1, R9.2
- new net SCL: J2.4, J3.4, J4.4, R1.1, U1.2
- new net SCL1: J1.4, J5.4, J6.4, R5.1, U2.2
- new net SCL2: J7.4, J8.4, J9.4, R8.1, U3.2
- new net SCL3: J10.4, J11.4, J12.4, R11.1, U4.2
- new net SCL4: J13.4, J14.4, J15.4, R14.1, U5.2
- new net SCL5: J16.4, J17.4, J18.4, R17.1, U6.2
- new net SCL6: J19.4, J20.4, J21.4, R20.1, U7.2
- new net SCL7: J22.4, J23.4, J24.4, R23.1, U8.2
- new net SCL8: J25.4, J26.4, J27.4, R26.1, U9.2
- new net SDA: J2.3, J3.3, J4.3, R2.1, U1.3
- new net SDA1: J1.3, J5.3, J6.3, R6.1, U2.3
- new net SDA2: J7.3, J8.3, J9.3, R9.1, U3.3
- new net SDA3: J10.3, J11.3, J12.3, R12.1, U4.3
- new net SDA4: J13.3, J14.3, J15.3, R15.1, U5.3
- new net SDA5: J16.3, J17.3, J18.3, R18.1, U6.3
- new net SDA6: J19.3, J20.3, J21.3, R21.1, U7.3
- new net SDA7: J22.3, J23.3, J24.3, R24.1, U8.3
- new net SDA8: J25.3, J26.3, J27.3, R27.1, U9.3
Routing:
- net 3.3V6: track 0.00 -> 62.7 mm, vias 0 -> 4
- net 3.3V7: track 0.00 -> 62.7 mm, vias 0 -> 4
- net 3.3V: track 0.00 -> 62.7 mm, vias 0 -> 4
- net 3.3V8: track 0.00 -> 62.7 mm, vias 0 -> 4
- net 3.3V3: track 0.00 -> 62.7 mm, vias 0 -> 4
- net 3.3V1: track 0.00 -> 62.7 mm, vias 0 -> 4
- net 3.3V2: track 0.00 -> 62.7 mm, vias 0 -> 4
- net 3.3V4: track 0.00 -> 62.7 mm, vias 0 -> 4
- net 3.3V5: track 0.00 -> 62.7 mm, vias 0 -> 4
- net SDA8: track 0.00 -> 43.9 mm, vias 0 -> 2
- net SDA7: track 0.00 -> 43.9 mm, vias 0 -> 2
- net SDA6: track 0.00 -> 43.9 mm, vias 0 -> 2
- net SDA5: track 0.00 -> 43.9 mm, vias 0 -> 2
- net SDA4: track 0.00 -> 43.9 mm, vias 0 -> 2
- net SDA3: track 0.00 -> 43.9 mm, vias 0 -> 2
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- added copper zone on layer 1, net GND
- added copper zone on layer 16, net GND
- added copper zone on layer 1, net GND1
- added copper zone on layer 16, net GND1
- added copper zone on layer 1, net GND2
- added copper zone on layer 16, net GND2
- added copper zone on layer 1, net GND3
- added copper zone on layer 16, net GND3
- added copper zone on layer 1, net GND4
- added copper zone on layer 16, net GND4
- added copper zone on layer 1, net GND5
- added copper zone on layer 16, net GND5
- added copper zone on layer 1, net GND6
- added copper zone on layer 16, net GND6
- added copper zone on layer 1, net GND7
- added copper zone on layer 16, net GND7
- added copper zone on layer 1, net GND8
- added copper zone on layer 16, net GND8
Other:
- board outline added: 97.3 x 97.3 mm
- board text added: "Dimensions in inches"
- board text added: "X01"
- board text added: "v-score"

Commit message: Update production files
Parts:
- added C10, C11, C12, C13, C14, C15, C16, C17, C18, C19, C20, C21, C22, C23, C24, C25: 0.1uF, SparkFun-Capacitors:0603
- added D10, D11, D12, D13, D14, D15, D16, D17, D18, D19, D20, D21, D22, D23, D24, D25: RED, SparkFun-LED:LED-0603
- added J28, J30, J31, J33, J34, J36, J37, J39, J40, J42, J43, J45, J46, J48, J49, J51, J52, J54, J55, J57, J58, J60, J61, J63, J64, J66, J67, J69, J70, J72, J73, J75: (no value), SparkFun-Connectors:1X04_1MM_RA
- added J29, J32, J35, J38, J41, J44, J47, J50, J53, J56, J59, J62, J65, J68, J71, J74: PTH, SparkX:1X04_NO_SILK
- added JP100, JP106, JP107, JP113, JP114, JP120, JP121, JP127, JP128, JP134, JP135, JP141, JP142, JP148, JP149, JP155, JP156, JP162, JP163, JP169, JP170, JP64, JP65, JP71, JP72, JP78, JP79, JP85, JP86, JP92, JP93, JP99: STAND-OFF, SparkFun:STAND-OFF
- added JP101, JP102, JP103, JP104, JP108, JP109, JP110, JP111, JP115, JP116, JP117, JP118, JP122, JP123, JP124, JP125, JP129, JP130, JP131, JP132, JP136, JP137, JP138, JP139, JP143, JP144, JP145, JP146, JP150, JP151, JP152, JP153, JP157, JP158, JP159, JP160, JP164, JP165, JP166, JP167, JP171, JP172, JP173, JP174, JP66, JP67, JP68, JP69, JP73, JP74, JP75, JP76, JP80, JP81, JP82, JP83, JP87, JP88, JP89, JP90, JP94, JP95, JP96, JP97: FIDUCIALUFIDUCIAL, SparkFun:MICRO-FIDUCIAL
- added JP105, JP112, JP119, JP126, JP133, JP140, JP147, JP154, JP161, JP168, JP175, JP70, JP77, JP84, JP91, JP98: JUMPER-SMT_3_2-NC_TRACE_SILK, SparkFun-Jumpers:SMT-JUMPER_3_2-NC_TRACE_SILK
- added LOGO10, LOGO11, LOGO12, LOGO13, LOGO14, LOGO15, LOGO16, LOGO17, LOGO18, LOGO19, LOGO20, LOGO21, LOGO22, LOGO23, LOGO24, LOGO25: OSHW-LOGOMINI, SparkFun-Aesthetics:OSHW-LOGO-MINI
- added R28, R31, R34, R37, R40, R43, R46, R49, R52, R55, R58, R61, R64, R67, R70, R73: 1k, SparkFun-Resistors:0603
- added R29, R30, R32, R33, R35, R36, R38, R39, R41, R42, R44, R45, R47, R48, R50, R51, R53, R54, R56, R57, R59, R60, R62, R63, R65, R66, R68, R69, R71, R72, R74, R75: 2.2k, SparkFun-Resistors:0603
- added U$136, U$147, U$152, U$163, U$168, U$179, U$184, U$195, U$200, U$211, U$216, U$227, U$232, U$243, U$248, U$259, U$264, U$275, U$280, U$291, U$296, U$307, U$312, U$323, U$328, U$339, U$344, U$355, U$360, U$371, U$376, U$387, U$392: (no value), Labels-0_04:3#3V2
- added U$137, U$150, U$153, U$166, U$169, U$182, U$185, U$198, U$201, U$214, U$217, U$230, U$233, U$246, U$249, U$262, U$265, U$278, U$281, U$294, U$297, U$310, U$313, U$326, U$329, U$342, U$345, U$358, U$361, U$374, U$377, U$390, U$393: (no value), Labels-0_04:SDA8
- added U$138, U$149, U$154, U$165, U$170, U$181, U$186, U$197, U$202, U$213, U$218, U$229, U$234, U$245, U$250, U$261, U$266, U$277, U$282, U$293, U$298, U$309, U$314, U$325, U$330, U$341, U$346, U$357, U$362, U$373, U$378, U$389, U$394: (no value), Labels-0_04:SCL9
- added U$139, U$155, U$171, U$187, U$203, U$219, U$235, U$251, U$267, U$283, U$299, U$315, U$331, U$347, U$363, U$379, U$395: (no value), Labels-0_04:(PWR)
- added U$140, U$141, U$156, U$157, U$172, U$173, U$188, U$189, U$204, U$205, U$220, U$221, U$236, U$237, U$252, U$253, U$268, U$269, U$284, U$285, U$300, U$301, U$316, U$317, U$332, U$333, U$348, U$349, U$364, U$365, U$380, U$381, U$396, U$397: (no value), buzzard_labels:SHTC3_HUMIDITY1
- added U$142, U$158, U$174, U$190, U$206, U$222, U$238, U$254, U$270, U$286, U$302, U$318, U$334, U$350, U$366, U$382, U$398: (no value), Labels:I_SUPER2_C-()-03
- added U$143, U$144, U$159, U$160, U$175, U$176, U$191, U$192, U$207, U$208, U$223, U$224, U$239, U$240, U$255, U$256, U$271, U$272, U$287, U$288, U$303, U$304, U$319, U$320, U$335, U$336, U$351, U$352, U$367, U$368, U$383, U$384, U$399, U$400: (no value), SparkFun-Aesthetics:QWIIC_5.5MM
- added U$145, U$146, U$161, U$162, U$177, U$178, U$193, U$194, U$209, U$210, U$225, U$226, U$241, U$242, U$257, U$258, U$273, U$274, U$289, U$290, U$305, U$306, U$321, U$322, U$337, U$338, U$353, U$354, U$369, U$370, U$385, U$386: SPARKX-LOGO4, SparkX:SPARKX-MEDIUM
- added U$148, U$151, U$164, U$167, U$180, U$183, U$196, U$199, U$212, U$215, U$228, U$231, U$244, U$247, U$260, U$263, U$276, U$279, U$292, U$295, U$308, U$311, U$324, U$327, U$340, U$343, U$356, U$359, U$372, U$375, U$388, U$391: (no value), Labels-0_04:GND1
- added U10, U11, U12, U13, U14, U15, U16, U17, U18, U19, U20, U21, U22, U23, U24, U25: SHTC3, SHTC3:SHTC3
- U$100, U$55: device Labels-0_04:SCL9 -> Labels-0_04:GND1
- U$101: device Labels-0_04:(PWR) -> Labels-0_04:SCL9
- U$102, U$57: device Labels:QWIIC-LOGO-MEDIUM -> Labels-0_04:SDA8
- U$103, U$119: device buzzard_labels:SHTC3_HUMIDITY1 -> Labels-0_04:GND1
- U$104, U$88: device buzzard_labels:SHTC3_HUMIDITY1 -> Labels-0_04:3#3V2
- U$105: device Labels:I_SUPER2_C-()-03 -> Labels-0_04:SDA8
- U$106, U$122: value SPARKX-LOGO4 -> (none); device SparkX:SPARKX-MEDIUM -> Labels-0_04:SCL9
- U$107, U$91: value SPARKX-LOGO4 -> (none); device SparkX:SPARKX-MEDIUM -> Labels-0_04:(PWR)
- U$108, U$93: device Labels-0_04:3#3V2 -> buzzard_labels:SHTC3_HUMIDITY1
- U$109, U$124: device Labels-0_04:GND1 -> buzzard_labels:SHTC3_HUMIDITY1
- U$11, U$12, U$31, U$32, U$47: value SPARKX-LOGO4 -> (none); device SparkX:SPARKX-MEDIUM -> SparkFun-Aesthetics:QWIIC_5.5MM
- U$110: device Labels-0_04:SCL9 -> Labels:I_SUPER2_C-()-03
- U$111, U$96: device Labels-0_04:SDA8 -> SparkFun-Aesthetics:QWIIC_5.5MM
- U$112, U$127, U$64, U$79: device Labels-0_04:GND1 -> SparkFun-Aesthetics:QWIIC_5.5MM
- U$113, U$13, U$33, U$98: value (none) -> SPARKX-LOGO4; device Labels-0_04:3#3V2 -> SparkX:SPARKX-MEDIUM
- U$114, U$129, U$66, U$81: value (none) -> SPARKX-LOGO4; device Labels-0_04:SDA8 -> SparkX:SPARKX-MEDIUM
- U$115, U$15, U$20, U$35, U$40: device Labels-0_04:SCL9 -> Labels-0_04:3#3V2
- U$116, U$71: device Labels-0_04:(PWR) -> Labels-0_04:GND1
- U$117, U$24, U$42: device Labels:QWIIC-LOGO-MEDIUM -> Labels-0_04:SCL9
- U$118, U$134, U$73, U$89: device buzzard_labels:SHTC3_HUMIDITY1 -> Labels-0_04:SDA8
- U$120: device Labels:I_SUPER2_C-()-03 -> Labels-0_04:3#3V2
- U$121: value SPARKX-LOGO4 -> (none); device SparkX:SPARKX-MEDIUM -> Labels-0_04:SDA8
- U$123: device Labels-0_04:3#3V2 -> Labels-0_04:(PWR)
- U$125: device Labels-0_04:SCL9 -> buzzard_labels:SHTC3_HUMIDITY1
- U$126: device Labels-0_04:SDA8 -> Labels:I_SUPER2_C-()-03
- U$128, U$48, U$63: device Labels-0_04:3#3V2 -> SparkFun-Aesthetics:QWIIC_5.5MM
- U$130, U$50, U$65: value (none) -> SPARKX-LOGO4; device Labels-0_04:SCL9 -> SparkX:SPARKX-MEDIUM
- U$131, U$56: device Labels-0_04:(PWR) -> Labels-0_04:3#3V2
- U$132, U$87: device Labels:QWIIC-LOGO-MEDIUM -> Labels-0_04:GND1
- U$133, U$58, U$74: device buzzard_labels:SHTC3_HUMIDITY1 -> Labels-0_04:SCL9
- U$135: device Labels:I_SUPER2_C-()-03 -> Labels-0_04:GND1
- U$14, U$34, U$49, U$82, U$97: value (none) -> SPARKX-LOGO4; device Labels-0_04:GND1 -> SparkX:SPARKX-MEDIUM
- U$16, U$19, U$36, U$39, U$84: device Labels-0_04:SDA8 -> Labels-0_04:GND1
- U$17, U$37: device Labels-0_04:GND1 -> Labels-0_04:SCL9
- U$18, U$38: device Labels-0_04:3#3V2 -> Labels-0_04:SDA8
- U$23, U$41, U$86: device Labels-0_04:(PWR) -> Labels-0_04:SDA8
- U$25, U$43, U$59: device buzzard_labels:SHTC3_HUMIDITY1 -> Labels-0_04:(PWR)
- U$29: device Labels:QWIIC-LOGO-MEDIUM -> buzzard_labels:SHTC3_HUMIDITY1
- U$45, U$60: device Labels:I_SUPER2_C-()-03 -> buzzard_labels:SHTC3_HUMIDITY1
- U$46, U$62: value SPARKX-LOGO4 -> (none); device SparkX:SPARKX-MEDIUM -> Labels:I_SUPER2_C-()-03
- U$51, U$99: device Labels-0_04:SDA8 -> Labels-0_04:3#3V2
- U$53: device Labels-0_04:3#3V2 -> Labels-0_04:SCL9
- U$61, U$76, U$77, U$92: value SPARKX-LOGO4 -> (none); device SparkX:SPARKX-MEDIUM -> buzzard_labels:SHTC3_HUMIDITY1
- U$67: device Labels-0_04:GND1 -> Labels-0_04:3#3V2
- U$68: device Labels-0_04:3#3V2 -> Labels-0_04:GND1
- U$69: device Labels-0_04:SDA8 -> Labels-0_04:SCL9
- U$70: device Labels-0_04:SCL9 -> Labels-0_04:SDA8
- U$72: device Labels:QWIIC-LOGO-MEDIUM -> Labels-0_04:3#3V2
- U$75: device Labels:I_SUPER2_C-()-03 -> Labels-0_04:(PWR)
- U$78: device Labels-0_04:3#3V2 -> Labels:I_SUPER2_C-()-03
- U$80, U$95: device Labels-0_04:SCL9 -> SparkFun-Aesthetics:QWIIC_5.5MM
- U$90: device Labels:I_SUPER2_C-()-03 -> Labels-0_04:SCL9
- U$94: device Labels-0_04:GND1 -> Labels:I_SUPER2_C-()-03
- moved U$74 99.1 mm to (120.1, 1.52), flipped to the bottom, turned to 90 degrees
- moved U$56 94.2 mm to (89.2, 1.52), flipped to the bottom, turned to 90 degrees
- moved U$71 91.8 mm to (112.5, 1.52), flipped to the bottom, turned to 90 degrees
- moved U$60 89.9 mm to (96.8, 21.3), turned to 0 degrees
- moved U$58 88.0 mm to (94.2, 1.52), turned to 90 degrees
- moved U$53 86.8 mm to (94.2, 1.52), flipped to the top
- moved U$73 85.8 mm to (117.6, 1.52), turned to 90 degrees
- moved U$67 84.3 mm to (115.1, 1.52), flipped to the top
- moved U$69 84.3 mm to (120.1, 1.52), flipped to the top
- moved U$59 82.1 mm to (78.4, 7.75)
- moved C4 81.9 mm to (90.6, 14.2)
- moved C5 81.9 mm to (116.5, 14.2)
- moved D4 81.9 mm to (80.9, 6.10)
- moved D5 81.9 mm to (106.8, 6.10)
- moved J10 81.9 mm to (82.8, 12.7)
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Connections:
- new net 3.3V10: C11.1, J31.2, J32.2, J33.2, JP77.2, R31.2, U11.1
- new net 3.3V11: C12.1, J34.2, J35.2, J36.2, JP84.2, R34.2, U12.1
- new net 3.3V12: C13.1, J37.2, J38.2, J39.2, JP91.2, R37.2, U13.1
- new net 3.3V13: C14.1, J40.2, J41.2, J42.2, JP98.2, R40.2, U14.1
- new net 3.3V14: C15.1, J43.2, J44.2, J45.2, JP105.2, R43.2, U15.1
- new net 3.3V15: C16.1, J46.2, J47.2, J48.2, JP112.2, R46.2, U16.1
- new net 3.3V16: C17.1, J49.2, J50.2, J51.2, JP119.2, R49.2, U17.1
- new net 3.3V17: C18.1, J52.2, J53.2, J54.2, JP126.2, R52.2, U18.1
- new net 3.3V18: C19.1, J55.2, J56.2, J57.2, JP133.2, R55.2, U19.1
- new net 3.3V19: C20.1, J58.2, J59.2, J60.2, JP140.2, R58.2, U20.1
- new net 3.3V20: C21.1, J61.2, J62.2, J63.2, JP147.2, R61.2, U21.1
- new net 3.3V21: C22.1, J64.2, J65.2, J66.2, JP154.2, R64.2, U22.1
- new net 3.3V22: C23.1, J67.2, J68.2, J69.2, JP161.2, R67.2, U23.1
- new net 3.3V23: C24.1, J70.2, J71.2, J72.2, JP168.2, R70.2, U24.1
- new net 3.3V24: C25.1, J73.2, J74.2, J75.2, JP175.2, R73.2, U25.1
- new net 3.3V9: C10.1, J28.2, J29.2, J30.2, JP70.2, R28.2, U10.1
- new net GND10: C11.2, D11.C, J31.1, J32.1, J33.1, U11.4, U11.5
- new net GND11: C12.2, D12.C, J34.1, J35.1, J36.1, U12.4, U12.5
- new net GND12: C13.2, D13.C, J37.1, J38.1, J39.1, U13.4, U13.5
- new net GND13: C14.2, D14.C, J40.1, J41.1, J42.1, U14.4, U14.5
- new net GND14: C15.2, D15.C, J43.1, J44.1, J45.1, U15.4, U15.5
- new net GND15: C16.2, D16.C, J46.1, J47.1, J48.1, U16.4, U16.5
- new net GND16: C17.2, D17.C, J49.1, J50.1, J51.1, U17.4, U17.5
- new net GND17: C18.2, D18.C, J52.1, J53.1, J54.1, U18.4, U18.5
- new net GND18: C19.2, D19.C, J55.1, J56.1, J57.1, U19.4, U19.5
- new net GND19: C20.2, D20.C, J58.1, J59.1, J60.1, U20.4, U20.5
- new net GND20: C21.2, D21.C, J61.1, J62.1, J63.1, U21.4, U21.5
- new net GND21: C22.2, D22.C, J64.1, J65.1, J66.1, U22.4, U22.5
- new net GND22: C23.2, D23.C, J67.1, J68.1, J69.1, U23.4, U23.5
- new net GND23: C24.2, D24.C, J70.1, J71.1, J72.1, U24.4, U24.5
- new net GND24: C25.2, D25.C, J73.1, J74.1, J75.1, U25.4, U25.5
- new net GND9: C10.2, D10.C, J28.1, J29.1, J30.1, U10.4, U10.5
- new net N$28: D10.A, R28.1
- new net N$29: JP70.3, R29.2
- new net N$30: JP70.1, R30.2
- new net N$31: D11.A, R31.1
- new net N$32: JP77.3, R32.2
- new net N$33: JP77.1, R33.2
- new net N$34: D12.A, R34.1
- new net N$35: JP84.3, R35.2
- new net N$36: JP84.1, R36.2
- new net N$37: D13.A, R37.1
- new net N$38: JP91.3, R38.2
- new net N$39: JP91.1, R39.2
- new net N$40: D14.A, R40.1
- new net N$41: JP98.3, R41.2
- new net N$42: JP98.1, R42.2
- new net N$43: D15.A, R43.1
- new net N$44: JP105.3, R44.2
- new net N$45: JP105.1, R45.2
- new net N$46: D16.A, R46.1
- new net N$47: JP112.3, R47.2
- new net N$48: JP112.1, R48.2
- new net N$49: D17.A, R49.1
- new net N$50: JP119.3, R50.2
- new net N$51: JP119.1, R51.2
- new net N$52: D18.A, R52.1
- new net N$53: JP126.3, R53.2
- new net N$54: JP126.1, R54.2
- new net N$55: D19.A, R55.1
- new net N$56: JP133.3, R56.2
- new net N$57: JP133.1, R57.2
- new net N$58: D20.A, R58.1
- new net N$59: JP140.3, R59.2
- new net N$60: JP140.1, R60.2
- new net N$61: D21.A, R61.1
- new net N$62: JP147.3, R62.2
- new net N$63: JP147.1, R63.2
- new net N$64: D22.A, R64.1
- new net N$65: JP154.3, R65.2
- new net N$66: JP154.1, R66.2
- new net N$67: D23.A, R67.1
- new net N$68: JP161.3, R68.2
- new net N$69: JP161.1, R69.2
- new net N$70: D24.A, R70.1
- new net N$71: JP168.3, R71.2
- new net N$72: JP168.1, R72.2
- new net N$73: D25.A, R73.1
- new net N$74: JP175.3, R74.2
- new net N$75: JP175.1, R75.2
- new net SCL10: J31.4, J32.4, J33.4, R32.1, U11.2
- new net SCL11: J34.4, J35.4, J36.4, R35.1, U12.2
- new net SCL12: J37.4, J38.4, J39.4, R38.1, U13.2
- new net SCL13: J40.4, J41.4, J42.4, R41.1, U14.2
- new net SCL14: J43.4, J44.4, J45.4, R44.1, U15.2
- new net SCL15: J46.4, J47.4, J48.4, R47.1, U16.2
- new net SCL16: J49.4, J50.4, J51.4, R50.1, U17.2
- new net SCL17: J52.4, J53.4, J54.4, R53.1, U18.2
- new net SCL18: J55.4, J56.4, J57.4, R56.1, U19.2
- new net SCL19: J58.4, J59.4, J60.4, R59.1, U20.2
- new net SCL20: J61.4, J62.4, J63.4, R62.1, U21.2
- new net SCL21: J64.4, J65.4, J66.4, R65.1, U22.2
- new net SCL22: J67.4, J68.4, J69.4, R68.1, U23.2
- new net SCL23: J70.4, J71.4, J72.4, R71.1, U24.2
- new net SCL24: J73.4, J74.4, J75.4, R74.1, U25.2
- new net SCL9: J28.4, J29.4, J30.4, R29.1, U10.2
- new net SDA10: J31.3, J32.3, J33.3, R33.1, U11.3
- new net SDA11: J34.3, J35.3, J36.3, R36.1, U12.3
- new net SDA12: J37.3, J38.3, J39.3, R39.1, U13.3
- new net SDA13: J40.3, J41.3, J42.3, R42.1, U14.3
- new net SDA14: J43.3, J44.3, J45.3, R45.1, U15.3
- new net SDA15: J46.3, J47.3, J48.3, R48.1, U16.3
- new net SDA16: J49.3, J50.3, J51.3, R51.1, U17.3
- new net SDA17: J52.3, J53.3, J54.3, R54.1, U18.3
- new net SDA18: J55.3, J56.3, J57.3, R57.1, U19.3
- new net SDA19: J58.3, J59.3, J60.3, R60.1, U20.3
- new net SDA20: J61.3, J62.3, J63.3, R63.1, U21.3
- new net SDA21: J64.3, J65.3, J66.3, R66.1, U22.3
- new net SDA22: J67.3, J68.3, J69.3, R69.1, U23.3
- new net SDA23: J70.3, J71.3, J72.3, R72.1, U24.3
- new net SDA24: J73.3, J74.3, J75.3, R75.1, U25.3
- new net SDA9: J28.3, J29.3, J30.3, R30.1, U10.3
Routing:
- net 3.3V10: track 0.00 -> 62.7 mm, vias 0 -> 4
- net 3.3V15: track 0.00 -> 62.7 mm, vias 0 -> 4
- net 3.3V18: track 0.00 -> 62.7 mm, vias 0 -> 4
- net 3.3V13: track 0.00 -> 62.7 mm, vias 0 -> 4
- net 3.3V11: track 0.00 -> 62.7 mm, vias 0 -> 4
- net 3.3V12: track 0.00 -> 62.7 mm, vias 0 -> 4
- net 3.3V19: track 0.00 -> 62.7 mm, vias 0 -> 4
- net 3.3V17: track 0.00 -> 62.7 mm, vias 0 -> 4
- net 3.3V16: track 0.00 -> 62.7 mm, vias 0 -> 4
- net 3.3V14: track 0.00 -> 62.7 mm, vias 0 -> 4
- net 3.3V20: track 0.00 -> 62.7 mm, vias 0 -> 4
- net 3.3V23: track 0.00 -> 62.7 mm, vias 0 -> 4
- net 3.3V21: track 0.00 -> 62.7 mm, vias 0 -> 4
- net 3.3V9: track 0.00 -> 62.7 mm, vias 0 -> 4
- net 3.3V24: track 0.00 -> 62.7 mm, vias 0 -> 4
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- added copper zone on layer 1, net GND10
- added copper zone on layer 16, net GND10
- added copper zone on layer 1, net GND11
- added copper zone on layer 16, net GND11
- added copper zone on layer 1, net GND12
- added copper zone on layer 16, net GND12
- added copper zone on layer 1, net GND13
- added copper zone on layer 16, net GND13
- added copper zone on layer 1, net GND14
- added copper zone on layer 16, net GND14
- added copper zone on layer 1, net GND15
- added copper zone on layer 16, net GND15
- added copper zone on layer 1, net GND16
- added copper zone on layer 16, net GND16
- added copper zone on layer 1, net GND17
- added copper zone on layer 16, net GND17
- added copper zone on layer 1, net GND18
- added copper zone on layer 16, net GND18
- added copper zone on layer 1, net GND19
- added copper zone on layer 16, net GND19
- added copper zone on layer 1, net GND20
- added copper zone on layer 16, net GND20
- added copper zone on layer 1, net GND21
- added copper zone on layer 16, net GND21
- added copper zone on layer 1, net GND22
- added copper zone on layer 16, net GND22
- added copper zone on layer 1, net GND23
- added copper zone on layer 16, net GND23
- added copper zone on layer 1, net GND24
- added copper zone on layer 16, net GND24
- added copper zone on layer 1, net GND9
- added copper zone on layer 16, net GND9
Other:
- board size 97.3 x 97.3 mm -> 149.1 x 149.1 mm
- board text added: "x02"
- board text removed: "Dimensions in inches"
- board text removed: "X01"
